File: openSX70_SCHEMATIC_COMPLETE.sch (EAGLE design)
At the start: 41 parts, among them Q1 5.8A/30V/35mΩ, Q2 5.8A/30V/35mΩ, U1 ATMEGA328P_TQFP, U3 BH1750FVI-TR, Y1 16MHz

Commit message: Eagle openSX70 pcb layout 2.0
Layout 2.0
Parts:
- FTDI: value (none) -> FTDI HEADER
- S1+, S1-, S2+, S2-, SOL2+, SOL2-: value SX70_S-PAD -> SX70-S-PAD-NEW; device openSX70:SX70_S-PAD -> openSX70:SX70-S-PAD-NEW
- renumbered BUZZ1 to BUZZER, J1 to FTDI, U3 to BH1750
Connections:
- net BUZZER: now also BUZZER.+
- net GND: now also BUZZER.-
Other:
- note added: "v 1.2B"
- note removed: "v 1.1B"
- moved on the sheet: C5, R12
