File: openSX70_SCHEMATIC_COMPLETE_NEW_LAYOUT_20171216.sch (EAGLE design)
At the start: 39 parts, among them Q1 5.8A/30V/35mΩ, Q2 5.8A/30V/35mΩ, U1 ATMEGA328P_TQFP, U3 BH1750FVI-TR, Y1 CSTCE16M0V53-R0

Commit message: Changed MOTOR pin from 19 to 25. The board is a mess and I have to start over.
Connections:
- removed net MOTOR+: R7.1, U1.ADC7
- new net MOTOR: R7.1, U1.PC2(ADC2)
Changed lines of the file:
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@@
-</segment>
-</net>
-<net name="MOTOR+" class="0">
-<segment>
-<pinref part="U1" gate="U$1" pin="ADC7"/>
-<wire x1="193.04" y1="109.22" x2="205.74" y2="109.22" width="0.1524" layer="91"/>
-<label x="195.58" y="109.22" size="1.778" layer="95"/>
-<pinref part="R7" gate="G$1" pin="1"/>
 </segment>
 </net>
@@
 </segment>
 </net>
+<net name="MOTOR" class="0">
+<segment>
+<pinref part="U1" gate="U$1" pin="PC2(ADC2)"/>
+<wire x1="193.04" y1="121.92" x2="205.74" y2="121.92" width="0.1524" layer="91"/>
+<pinref part="R7" gate="G$1" pin="1"/>
+<wire x1="205.74" y1="121.92" x2="205.74" y2="109.22" width="0.1524" layer="91"/>
+<label x="195.58" y="121.92" size="1.778" layer="95"/>
+</segment>
+</net>
