File: openSX70_WIP_NEW_LAYOUT_20171220.brd (EAGLE design)
At the start: 95.9 x 27.9 mm, 39 parts, among them Q1 5.8A/30V/35mΩ, Q2 5.8A/30V/35mΩ, U1 ATMEGA328P_TQFP, U3 BH1750FVI-TR, Y1 CSTCE16M0V53-R0

Commit message: minor updates in new layout. Routing manually important traces.
Parts:
- removed R15, R16: 4K7, resistor:R0603
- moved U1 110.7 mm to (81.2, 15.7), turned to 45 degrees
- moved CONN1 73.9 mm to (41.3, 15.9)
- moved U3 63.3 mm to (18.8, 20.3), turned to 270 degrees
- moved LED1 46.3 mm to (19.7, 4.45), flipped to the bottom
- moved LD11173.3V 37.9 mm to (7.62, 10.2), turned to 180 degrees
- moved BUZZ1 30.6 mm to (12.8, 6.48), flipped to the bottom, turned to 90 degrees
Connections:
- net 3.3V: no longer R15.1, R16.1
- net SCL: no longer R15.2
- net SDA: no longer R16.2
Routing:
- net 6V: track 0.00 -> 23.8 mm, vias 0 -> 2
- net GND: track 0.00 -> 10.2 mm
- net S2: track 0.00 -> 5.74 mm

Commit message: Painfully laying out components and routing, manually.
Parts:
- moved Q1 130.9 mm to (86.4, 8.89), turned to 90 degrees
- moved Y1 129.4 mm to (77.2, 9.40), turned to 315 degrees
- moved R7 127.5 mm to (85.6, 25.8)
- moved R9 109.4 mm to (71.8, 23.5), turned to 180 degrees
- moved R6 100.9 mm to (67.9, 21.6), turned to 180 degrees
- moved R5 99.6 mm to (71.8, 21.6)
- moved D1 99.3 mm to (76.7, 26.0), turned to 90 degrees
- moved R10 97.5 mm to (67.9, 23.5), turned to 180 degrees
- moved C6 97.1 mm to (73.7, 8.26)
- moved Q2 84.5 mm to (68.6, 8.26), turned to 270 degrees
- moved C7 74.9 mm to (22.2, 13.3)
- moved R8 70.1 mm to (19.7, 8.26), flipped to the bottom, turned to 90 degrees
- moved C5 62.8 mm to (15.2, 18.6), flipped to the bottom
- moved C2 62.6 mm to (14.6, 12.7)
- moved R14 60.4 mm to (15.2, 22.2), flipped to the bottom
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Routing:
- net 3.3V: track 0.00 -> 91.8 mm, vias 0 -> 4
- net 6V: track 23.8 -> 101.3 mm
- net MOTOR-HEADER: track 0.00 -> 23.0 mm, vias 0 -> 2
- net S9@6V: track 0.00 -> 9.41 mm, vias 0 -> 1
- net MOTOR+: track 0.00 -> 8.02 mm, vias 0 -> 2
- net S8@6V: track 0.00 -> 7.47 mm, vias 0 -> 1
- net SOL2-: track 0.00 -> 4.15 mm
- net S1: track 0.00 -> 2.83 mm
- net GND: vias 0 -> 1
