File: openSX70_WIP_NEW_LAYOUT_20171229_V30_manually-routed-pre-AR.brd (EAGLE design)
At the start: 95.9 x 27.9 mm, 37 parts, among them Q1 5.8A/30V/35mΩ, Q2 5.8A/30V/35mΩ, U1 ATMEGA328P_TQFP, U3 BH1750FVI-TR, Y1 CSTCE16M0V53-R0

Commit message: V3.2  added license text. Will do to all brd.
Parts:
- moved R6 18.5 mm to (70.5, 19.6), turned to 0 degrees
- moved R5 18.1 mm to (66.9, 19.6), turned to 0 degrees
- moved R10 16.8 mm to (70.5, 21.8), turned to 0 degrees
- moved R9 16.5 mm to (66.9, 21.8), turned to 0 degrees
- moved C5 0.19 mm to (15.2, 18.4)
- moved R14 0.16 mm to (15.2, 22.4)
Routing:
- net S9@6V: track 23.7 -> 61.6 mm, vias 1 -> 4
- net S8@6V: track 19.7 -> 51.7 mm, vias 1 -> 2
- net S8@3.3V: track 5.66 -> 17.7 mm, vias 1 -> 2
- net S9@3.3V: track 7.00 -> 18.5 mm, vias 1 -> 2
- net N$26: track 5.34 -> 0.00 mm
- net 3.3V: track 151.8 -> 149.7 mm
- net S5: track 14.5 -> 16.1 mm
- net GND: track 16.7 -> 18.2 mm
- net SOL1-: track 12.7 -> 11.8 mm
- net S2: track 5.74 -> 4.85 mm
- net S3: track 14.5 -> 13.9 mm
