File: openSX70_WIP_NEW_LAYOUT_20171230_V30_manually-routed-pre-AR.brd (EAGLE design)
At the start: 95.9 x 27.9 mm, 37 parts, among them Q1 5.8A/30V/35mΩ, Q2 5.8A/30V/35mΩ, U1 ATMEGA328P_TQFP, U3 BH1750FVI-TR, Y1 CSTCE16M0V53-R0

Commit message: V3.2  added license text. Will do to all brd.
Parts:
- moved R10 27.8 mm to (26.4, 21.7), turned to 180 degrees
- moved R6 27.6 mm to (26.0, 17.0), turned to 180 degrees
- moved R5 25.7 mm to (24.5, 14.1), turned to 180 degrees
- moved R9 22.8 mm to (28.0, 19.5), turned to 180 degrees
- moved CONN1 7.33 mm to (28.9, 5.08), turned to 0 degrees
- moved R4 1.98 mm to (71.6, 22.7), turned to 90 degrees
- moved C7 1.42 mm to (69.8, 17.8)
- moved R3 1.41 mm to (68.6, 22.7), turned to 90 degrees
- moved C5 0.19 mm to (15.2, 18.4)
- moved R14 0.16 mm to (15.2, 22.4)
Routing:
- net S9@6V: track 23.7 -> 113.4 mm, vias 1 -> 6
- net S8@6V: track 19.7 -> 92.5 mm, vias 1 -> 2
- net S9@3.3V: track 7.00 -> 76.1 mm, vias 1 -> 4
- net S8@3.3V: track 5.66 -> 69.1 mm, vias 1 -> 4
- net SCL: track 0.00 -> 52.4 mm, vias 0 -> 1
- net SDA: track 0.00 -> 52.3 mm, vias 0 -> 1
- net DTR: track 0.00 -> 46.7 mm
- net 6V: track 122.9 -> 141.5 mm
- net FF: track 68.6 -> 85.3 mm
- net TXD: track 0.00 -> 16.6 mm
- net RXD: track 0.00 -> 13.7 mm
- net S1: track 2.83 -> 13.3 mm, vias 0 -> 2
- net N$26: track 5.34 -> 0.00 mm
- net S2: track 5.74 -> 8.66 mm
- net 3.3V: track 151.8 -> 154.3 mm
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