File: openSX70_WIP_NEW_LAYOUT_20171230_V31_manually-routed-AR.brd (EAGLE design)
At the start: 95.9 x 27.9 mm, 37 parts, among them Q1 5.8A/30V/35mΩ, Q2 5.8A/30V/35mΩ, U1 ATMEGA328P_TQFP, U3 BH1750FVI-TR, Y1 CSTCE16M0V53-R0

Commit message: V3.2  added license text. Will do to all brd.
Parts:
- BUZZ1: device CSET8-5G_B:CSET8-5G_PACKAGE -> openSX70:CSET8-5G_PACKAGE
- moved R10 27.8 mm to (26.4, 21.7), turned to 180 degrees
- moved R6 27.6 mm to (26.0, 17.0), turned to 180 degrees
- moved R5 25.7 mm to (24.5, 14.1), turned to 180 degrees
- moved R9 22.8 mm to (28.0, 19.5), turned to 180 degrees
- moved CONN1 7.33 mm to (28.9, 5.08), turned to 0 degrees
- moved R4 1.98 mm to (71.6, 22.7), turned to 90 degrees
- moved C7 1.42 mm to (69.8, 17.8)
- moved R3 1.41 mm to (68.6, 22.7), turned to 90 degrees
- moved C5 0.19 mm to (15.2, 18.4)
- moved R14 0.16 mm to (15.2, 22.4)
Connections:
- net GND: now also BUZZ1.GND; no longer BUZZ1.GND-
Routing:
- net SDA: track 0.00 -> 105.7 mm, vias 0 -> 3
- net S9@6V: track 23.7 -> 113.7 mm, vias 1 -> 6
- net SCL: track 0.00 -> 79.1 mm, vias 0 -> 3
- net S9@3.3V: track 7.00 -> 80.1 mm, vias 1 -> 4
- net S8@6V: track 19.7 -> 92.4 mm, vias 1 -> 2
- net S8@3.3V: track 5.66 -> 74.9 mm, vias 1 -> 4
- net DTR: track 0.00 -> 63.7 mm, vias 0 -> 1
- net RXD: track 0.00 -> 60.0 mm, vias 0 -> 1
- net TXD: track 0.00 -> 51.2 mm, vias 0 -> 2
- net 6V: track 122.9 -> 172.4 mm, vias 3 -> 4
- net GND: track 16.7 -> 62.3 mm, vias 6 -> 31
- net SOL2: track 0.00 -> 25.8 mm, vias 0 -> 2
- net 3.3V: track 151.8 -> 174.0 mm, vias 6 -> 7
- net N$9: track 0.00 -> 19.0 mm
- net FF: track 68.6 -> 87.2 mm
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Other:
- board text added: "20180102"
- board text added: "3.3V"
- board text added: "6V"
- board text added: "BUZZER"
- board text added: "Creative Commons "Attribution-NonCommercial 4.0 International (CC BY-NC 4.0)" https://creativecommons.org/licenses/by-nc/4.0/"
- board text added: "DTR"
- board text added: "F+"
- board text added: "F-"
- board text added: "FF"
- board text added: "FT"
- board text added: "FTDI HEADER"
- board text added: "GND"
- board text added: "LIGHT METER"
- board text added: "MOTOR"
- board text added: "RXD"
- board text added: "S1+"
- board text added: "S1-"
- board text added: "S2+"
- board text added: "S2-"
- board text added: "S3"
- board text added: "S5"
- board text added: "S8"
- board text added: "S9"
- board text added: "SOL1+"
- board text added: "SOL1-"
- board text added: "SOL2+"
- board text added: "SOL2-"
- board text added: "TXD"
- board text added: "VCC"
- board text added: "layout 3.1"
- board text added: "www.openSX70.com"
