File: openSX70_chocolate_V34_20180103_manually-routed-and-AR.brd (EAGLE design)
At the start: 95.9 x 27.9 mm, 37 parts, among them Q1 5.8A/30V/35mΩ, Q2 5.8A/30V/35mΩ, U1 ATMEGA328P_TQFP, U3 BH1750FVI-TR, Y1 CSTCE16M0V53-R0

Commit message: More cosmetic stuff.
Routing:
- net LED: track 94.1 -> 92.9 mm
Changed lines of the file:
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@@
 <wire x1="84.9359375" y1="6.48540625" x2="84.93595" y2="6.4877375" width="0.254" layer="16"/>
 <wire x1="83.82" y1="5.3717875" x2="84.72074375" y2="6.27253125" width="0.254" layer="16"/>
-<wire x1="84.93595" y1="6.4877375" x2="85.59498125" y2="7.14676875" width="0.254" layer="16"/>
-<wire x1="85.59498125" y1="7.14676875" x2="91.821" y2="7.20725" width="0.254" layer="16"/>
-<wire x1="91.821" y1="7.20725" x2="91.3765" y2="8.98525" width="0.254" layer="16"/>
+<wire x1="84.93595" y1="6.4877375" x2="85.46798125" y2="7.01976875" width="0.254" layer="16"/>
+<wire x1="85.46798125" y1="7.01976875" x2="90.424" y2="7.08025" width="0.254" layer="16"/>
+<wire x1="90.424" y1="7.08025" x2="91.3765" y2="8.98525" width="0.254" layer="16"/>
 <wire x1="87.34425" y1="16.898675" x2="88.48725" y2="15.77975" width="0.254" layer="1"/>
 <wire x1="88.48725" y1="15.77975" x2="88.52423125" y2="15.59448125" width="0.254" layer="1"/>
