File: CURRENT/openSX70_ALADDIN_V395SEEED_20180208.brd (EAGLE design)
At the start: 95.9 x 27.9 mm, 42 parts, among them J1 GND, Q1 2N7002, Q2 2N7002, U1 ATMEGA328P_TQFP, U3 BH1750FVI-TR, Y1 CSTCE8M00G52Z-R0

Commit message: working on a manufacturable version
Routing:
- net GND: track 38.4 -> 35.5 mm
Changed lines of the file:
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@@
 METER</text>
 <text x="15.08125" y="4.92125" size="0.8128" layer="22" font="vector" ratio="20" rot="MR0">BUZZER</text>
-<text x="10.7315" y="25.019" size="0.6096" layer="21" font="vector" ratio="20" rot="R90">DTR</text>
-<text x="11.46175" y="24.9555" size="0.6096" layer="21" font="vector" ratio="20" rot="R90">TXD</text>
-<text x="12.09675" y="24.98725" size="0.6096" layer="21" font="vector" ratio="20" rot="R90">RXD</text>
-<text x="12.79525" y="24.98725" size="0.6096" layer="21" font="vector" ratio="20" rot="R90">VCC</text>
-<text x="13.843" y="24.86025" size="0.6096" layer="21" font="vector" ratio="20" rot="R90">GND</text>
+<text x="10.541" y="24.765" size="0.7112" layer="21" font="vector" ratio="10" rot="R90">DTR</text>
+<text x="11.39825" y="24.7015" size="0.7112" layer="21" font="vector" ratio="10" rot="R90">TXD</text>
+<text x="12.16025" y="24.73325" size="0.7112" layer="21" font="vector" ratio="10" rot="R90">RXD</text>
+<text x="12.98575" y="24.73325" size="0.7112" layer="21" font="vector" ratio="10" rot="R90">VCC</text>
+<text x="14.097" y="24.66975" size="0.7112" layer="21" font="vector" ratio="10" rot="R90">GND</text>
 <text x="13.55725" y="6.5405" size="0.8128" layer="21" font="vector" ratio="20" rot="R90">GND</text>
 <text x="13.55725" y="12.1285" size="0.8128" layer="21" font="vector" ratio="20" rot="R90">6V</text>
@@
 <text x="10.4775" y="15.748" size="0.8128" layer="21" font="vector" ratio="20" rot="R90">6V</text>
 <text x="10.4775" y="18.161" size="0.8128" layer="21" font="vector" ratio="20" rot="R90">2.5V</text>
-<text x="27.305" y="11.1125" size="0.8128" layer="21" font="vector" ratio="20">VCC</text>
-<text x="29.337" y="5.6515" size="0.8128" layer="21" font="vector" ratio="20" rot="R180">MISO</text>
-<text x="34.163" y="5.6515" size="0.8128" layer="21" font="vector" ratio="20" rot="R180">RST</text>
-<text x="31.623" y="5.6515" size="0.8128" layer="21" font="vector" ratio="20" rot="R180">SCK</text>
-<text x="29.464" y="11.1125" size="0.8128" layer="21" font="vector" ratio="20">MOSI</text>
-<text x="32.258" y="11.1125" size="0.8128" layer="21" font="vector" ratio="20">GND</text>
+<text x="28.5115" y="11.303" size="0.8128" layer="21" font="vector" ratio="20" rot="R90">VCC</text>
+<text x="27.686" y="5.461" size="0.8128" layer="21" font="vector" ratio="20" rot="R270">MISO</text>
+<text x="32.8295" y="5.207" size="0.8128" layer="21" font="vector" ratio="20" rot="R270">RST</text>
+<text x="30.353" y="5.334" size="0.8128" layer="21" font="vector" ratio="20" rot="R270">SCK</text>
+<text x="31.0515" y="11.176" size="0.8128" layer="21" font="vector" ratio="20" rot="R90">MOSI</text>
+<text x="33.3375" y="11.303" size="0.8128" layer="21" font="vector" ratio="20" rot="R90">GND</text>
 <circle x="26.67" y="5.842" radius="0.1419875" width="0.3048" layer="21"/>
 </plain>
@@
 </polygon>
 <contactref element="Y1" pad="GND"/>
-<wire x1="23.1648" y1="23.368" x2="22.5552" y2="23.368" width="0.2032" layer="1"/>
-<wire x1="24.7904" y1="24.9936" x2="23.1648" y2="23.368" width="0.2032" layer="1"/>
 <wire x1="24.7904" y1="24.9936" x2="24.9682" y2="25.146" width="0.2032" layer="1"/>
 <wire x1="77.6224" y1="21.5392" x2="74.3712" y2="21.5392" width="0.2032" layer="16"/>
@@
 <wire x1="81.0768" y1="10.3632" x2="82.7024" y2="11.9888" width="0.2032" layer="16"/>
 <wire x1="73.5584" y1="10.3632" x2="81.0768" y2="10.3632" width="0.2032" layer="16"/>
-<via x="22.5552" y="23.368" extent="1-16" drill="0.35"/>
+<via x="22.2377" y="22.098" extent="1-16" drill="0.35"/>
 <via x="74.3712" y="21.5392" extent="1-16" drill="0.35"/>
 <via x="77.6224" y="21.5392" extent="1-16" drill="0.35"/>
