File: CURRENT/openSX70_ALADDIN_V398SEEED_20180219.sch (EAGLE design)
At the start: 46 parts, among them Q1 5.8A/30V/35mΩ, Q2 5.8A/30V/35mΩ, Q3 MMBT3904LT1G, U1 ATMEGA328P_TQFP, U3 BH1750FVI-TR, Y1 CSTCE8M00G52Z-R0

Commit message: Updated to 8.6.3 eagle and more
Other:
- note added: "v 3.9.8S"
- note removed: "v 3.9.5S"
- moved on the sheet: R7
Changed lines of the file:
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@@
 <?xml version="1.0" encoding="utf-8"?>
 <!DOCTYPE eagle SYSTEM "eagle.dtd">
-<eagle version="8.6.1">
+<eagle version="8.6.3">
 <drawing>
 <settings>
@@
 or
 FLASH</text>
-<text x="246.38" y="2.54" size="2.1844" layer="97" align="center">v 3.9.5S</text>
+<text x="246.38" y="2.54" size="2.1844" layer="97" align="center">v 3.9.8S</text>
 <text x="203.454" y="24.638" size="2.0066" layer="97" align="center">Design by Joaquín de Prada
 Creative Commons "Attribution-NonCommercial 4.0 International (CC BY-NC 4.0)"
@@
 <attribute name="VALUE" x="76.454" y="59.944" size="1.778" layer="96"/>
 </instance>
-<instance part="R7" gate="G$1" x="210.82" y="109.22"/>
+<instance part="R7" gate="G$1" x="212.09" y="121.92"/>
 <instance part="R8" gate="G$1" x="27.94" y="7.62" rot="R90"/>
 <instance part="GND8" gate="1" x="88.9" y="63.5" rot="R90"/>
@@
 </instance>
 <instance part="GND13" gate="1" x="-6.604" y="53.086" rot="R180"/>
-<instance part="U$4" gate="G$1" x="137.16" y="15.24" rot="MR180"/>
+<instance part="U$4" gate="G$1" x="137.16" y="15.24" smashed="yes" rot="MR180">
+<attribute name="VALUE" x="115.57" y="4.572" size="1.27" layer="96" rot="MR180"/>
+</instance>
 <instance part="R15" gate="G$1" x="-1.778" y="39.116" smashed="yes">
 <attribute name="NAME" x="-5.588" y="41.1226" size="1.778" layer="95"/>
@@
 <wire x1="228.6" y1="93.98" x2="215.9" y2="93.98" width="0.1524" layer="91"/>
 <pinref part="R7" gate="G$1" pin="2"/>
-<wire x1="214.63" y1="109.22" x2="215.9" y2="93.98" width="0.1524" layer="91"/>
+<wire x1="215.9" y1="121.92" x2="215.9" y2="93.98" width="0.1524" layer="91"/>
 </segment>
 </net>
@@
 <segment>
 <pinref part="U1" gate="U$1" pin="PC2(ADC2)"/>
-<wire x1="193.04" y1="121.92" x2="205.74" y2="121.92" width="0.1524" layer="91"/>
+<wire x1="193.04" y1="121.92" x2="208.28" y2="121.92" width="0.1524" layer="91"/>
 <pinref part="R7" gate="G$1" pin="1"/>
-<wire x1="205.74" y1="121.92" x2="207.01" y2="109.22" width="0.1524" layer="91"/>
 <label x="195.58" y="121.92" size="1.778" layer="95"/>
 </segment>
