File: CURRENT/openSX70_ALPHA_V6.2-20181009.brd (EAGLE design)
At the start: 95.9 x 27.9 mm, 38 parts, among them J1 687106183722, Q1 5.8A/30V/35mΩ, Q2 5.8A/30V/35mΩ, U1 ATMEGA328P_TQFP, Y1 CSTCE8M00G52Z-R0

Commit message: wip
Parts:
- added SOL2: SX70-SOLENOID1-2PADS, openSX70:SX70-SOLENOID1-2
Routing:
- net 6V: track 188.1 -> 195.7 mm, vias 5 -> 7
- net SOL2: track 90.1 -> 86.0 mm, vias 6 -> 4
- net FF: track 69.5 -> 67.2 mm
Changed lines of the file:
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@@
 <element name="R7" library="Seeed-Resistor" library_urn="urn:adsk.eagle:library:474" package="R0603" package3d_urn="urn:adsk.eagle:package:32791/1" value="100R" x="87.6005" y="25.456" rot="R90">
 <attribute name="MPN" value="RC0603JR-07100RL" x="87.6005" y="25.456" size="1.778" layer="27" rot="R90" display="off"/>
-<attribute name="NAME" x="91.727996875" y="25.932246875" size="0.8128" layer="25" font="vector" ratio="20" rot="R180"/>
+<attribute name="NAME" x="88.437996875" y="24.437246875" size="0.8128" layer="25" font="vector" ratio="20" rot="R180"/>
 <attribute name="VALUE" value="100R" x="87.8545" y="27.868996875" size="0.8128" layer="27" font="vector" rot="R90"/>
 </element>
@@
 <attribute name="NAME" x="13.569" y="16.775" size="0.635" layer="33" ratio="10" rot="R90"/>
 <attribute name="VALUE" x="14.9025" y="16.775" size="0.635" layer="27" ratio="10" rot="R90"/>
+</element>
+<element name="SOL2" library="openSX70" package="SX70-SOLENOID1-2" value="SX70-SOLENOID1-2PADS" x="77.555" y="4.7835">
+<attribute name="NAME" x="76.031" y="6.1805" size="0.4064" layer="21"/>
 </element>
 </elements>
@@
 <via x="67.31" y="23.8125" extent="1-16" drill="0.35"/>
 <via x="85.05825" y="16.54175" extent="1-16" drill="0.35"/>
-<wire x1="29.73705" y1="10.58545" x2="29.68625" y2="15.1003" width="0.4064" layer="16"/>
-<via x="29.68625" y="15.1003" extent="1-16" drill="0.35"/>
 <wire x1="67.31" y1="23.8125" x2="63.9445" y2="23.8125" width="0.254" layer="16"/>
 <wire x1="63.9445" y1="23.8125" x2="63.246" y2="24.511" width="0.254" layer="16"/>
@@
 <wire x1="29.0195" y1="26.162" x2="27.051" y2="24.003" width="0.254" layer="1"/>
 <via x="27.051" y="24.003" extent="1-16" drill="0.35"/>
-<wire x1="28.4508" y1="22.228025" x2="28.895525" y2="21.7833" width="0.254" layer="16"/>
-<wire x1="31.0487" y1="21.7833" x2="32.766" y2="20.066" width="0.254" layer="16"/>
-<wire x1="28.895525" y1="21.7833" x2="31.0487" y2="21.7833" width="0.254" layer="16"/>
-<wire x1="27.051" y1="24.003" x2="28.4508" y2="22.6032" width="0.254" layer="16"/>
-<wire x1="28.4508" y1="22.6032" x2="28.4508" y2="22.228025" width="0.254" layer="16"/>
-<via x="32.766" y="20.066" extent="1-16" drill="0.35"/>
-<wire x1="29.68625" y1="15.1003" x2="32.77235" y2="17.55775" width="0.254" layer="1"/>
-<wire x1="32.77235" y1="17.55775" x2="32.766" y2="20.066" width="0.254" layer="1"/>
 <contactref element="ICSP" pad="5"/>
-<wire x1="29.73705" y1="10.58545" x2="29.845" y2="10.4775" width="0.1524" layer="16"/>
-<wire x1="29.845" y1="10.4775" x2="30.7975" y2="9.7155" width="0.4064" layer="16"/>
 <wire x1="67.31" y1="23.8125" x2="68.5165" y2="23.8125" width="0.254" layer="1"/>
 <wire x1="68.5165" y1="23.8125" x2="68.707" y2="23.622" width="0.254" layer="1"/>
@@
 <wire x1="59.67095" y1="27.432" x2="62.12051875" y2="24.510325" width="0.254" layer="1"/>
 <wire x1="67.31" y1="23.8125" x2="77.70495" y2="23.7998" width="0.254" layer="16"/>
+<wire x1="27.051" y1="24.003" x2="27.051" y2="13.799" width="0.3048" layer="16"/>
+<wire x1="30.7975" y1="10.0525" x2="30.7975" y2="9.7155" width="0.3048" layer="16"/>
+<wire x1="27.051" y1="13.799" x2="30.7975" y2="10.0525" width="0.3048" layer="16"/>
 </signal>
 <signal name="FF">
@@
 <wire x1="63.11265" y1="22.2885" x2="62.865" y2="22.733" width="0.4064" layer="16"/>
 <via x="62.865" y="22.733" extent="1-16" drill="0.35"/>
-<wire x1="25.0825" y1="23.1775" x2="28.5115" y2="23.1775" width="0.4064" layer="1"/>
-<wire x1="28.5115" y1="23.1775" x2="30.607" y2="25.4" width="0.4064" layer="1"/>
+<wire x1="28.53035625" y1="23.1975" x2="30.607" y2="25.4" width="0.4064" layer="1"/>
 <contactref element="U1" pad="2"/>
 <wire x1="21.1836" y1="25.146" x2="21.209" y2="25.1206" width="0.4064" layer="1"/>
-<wire x1="21.1836" y1="25.146" x2="21.1836" y2="22.7076" width="0.4064" layer="1"/>
-<wire x1="21.1836" y1="22.7076" x2="21.209" y2="21.844" width="0.4064" layer="1"/>
-<wire x1="21.209" y1="21.844" x2="22.1615" y2="21.209" width="0.4064" layer="1"/>
-<wire x1="22.1615" y1="21.209" x2="23.3045" y2="21.209" width="0.4064" layer="1"/>
-<wire x1="23.3045" y1="21.209" x2="25.0825" y2="23.1775" width="0.4064" layer="1"/>
+<wire x1="21.1836" y1="25.146" x2="21.1336" y2="25.096" width="0.4064" layer="1"/>
+<wire x1="21.1336" y1="25.096" x2="21.1336" y2="23.1975" width="0.4064" layer="1"/>
+<wire x1="28.53035625" y1="23.1975" x2="21.1336" y2="23.1975" width="0.4064" layer="1"/>
 <wire x1="71.5391" y1="22.33295" x2="75.184" y2="18.415" width="0.4064" layer="16"/>
 <wire x1="75.184" y1="18.415" x2="75.7555" y2="18.415" width="0.4064" layer="16"/>
@@
 <wire x1="72.36625625" y1="4.4583" x2="72.422915625" y2="4.4583" width="1.016" layer="16"/>
 <wire x1="71.760259375" y1="4.43391875" x2="72.422915625" y2="4.4583" width="0.8128" layer="16"/>
-<wire x1="78.74" y1="4.7885" x2="81.661" y2="4.7885" width="1.016" layer="16"/>
 <wire x1="81.661" y1="4.7885" x2="83.947" y2="6.9215" width="1.016" layer="16"/>
-<wire x1="78.74" y1="4.7885" x2="77.216" y2="4.8111" width="0.8128" layer="16"/>
-<via x="77.216" y="4.8111" extent="1-16" drill="0.35"/>
-<wire x1="77.216" y1="4.8111" x2="80.01" y2="4.826" width="1.016" layer="1"/>
 <wire x1="80.01" y1="4.826" x2="80.264" y2="4.981" width="1.016" layer="1"/>
 <wire x1="93.499328125" y1="14.708528125" x2="93.7895" y2="14.986" width="0.8128" layer="1"/>
@@
 <wire x1="72.62025625" y1="4.69389375" x2="72.36625625" y2="4.4583" width="1.016" layer="16"/>
 <wire x1="74.676" y1="5.588" x2="73.5143625" y2="5.588" width="1.016" layer="16"/>
-<wire x1="78.74" y1="4.7885" x2="75.4755" y2="4.7885" width="1.016" layer="16"/>
+<wire x1="81.661" y1="4.7885" x2="75.4755" y2="4.7885" width="1.016" layer="16"/>
 <wire x1="75.4755" y1="4.7885" x2="74.676" y2="5.588" width="1.016" layer="16"/>
 <wire x1="80.5942" y1="5.45465" x2="80.01" y2="4.826" width="0.6096" layer="1"/>
 <wire x1="10.7188" y1="12.4714" x2="10.274478125" y2="12.746709375" width="0.8128" layer="1"/>
 <wire x1="10.274478125" y1="12.746709375" x2="10.287" y2="19.8755" width="0.8128" layer="1"/>
-<wire x1="80.264" y1="4.981" x2="80.2005" y2="6.0605" width="0.6096" layer="1"/>
-<wire x1="80.2005" y1="6.6245" x2="80.515" y2="7.239" width="0.6096" layer="1"/>
-<wire x1="80.2005" y1="6.0605" x2="80.2005" y2="6.6245" width="0.6096" layer="1"/>
+<wire x1="80.285790625" y1="6.791146875" x2="80.515" y2="7.239" width="0.6096" layer="1"/>
 <wire x1="10.0584" y1="16.6624" x2="8.5344" y2="16.6624" width="0.2032" layer="1"/>
 <wire x1="8.5344" y1="16.6624" x2="8.382" y2="16.637" width="0.2032" layer="1"/>
@@
 <wire x1="83.045946875" y1="19.635" x2="87.38" y2="19.635" width="0.6096" layer="16"/>
 <wire x1="83.045946875" y1="19.635" x2="83.04" y2="19.705" width="0.6096" layer="16"/>
+<wire x1="80.264" y1="4.981" x2="80.2005" y2="6.6245" width="1.016" layer="1"/>
+<wire x1="80.285790625" y1="6.791146875" x2="79.03168125" y2="8.13903125" width="1.016" layer="1"/>
+<wire x1="79.035" y1="8.185" x2="79.03168125" y2="8.13903125" width="1.016" layer="1"/>
+<via x="79.035" y="8.185" extent="1-16" drill="0.35"/>
+<wire x1="79.035" y1="8.185" x2="78.96" y2="8.26" width="1.016" layer="16"/>
+<wire x1="78.96" y1="8.26" x2="72.125" y2="8.26" width="1.016" layer="16"/>
+<via x="72.125" y="8.26" extent="1-16" drill="0.35"/>
+<wire x1="72.125" y1="8.26" x2="72.125" y2="6.9773625" width="1.016" layer="1"/>
+<wire x1="72.125" y1="6.9773625" x2="73.5143625" y2="5.588" width="1.016" layer="1"/>
+<via x="73.5143625" y="5.588" extent="1-16" drill="0.35"/>
 <wire x1="85.0817" y1="22.098" x2="85.109" y2="22.098" width="0" layer="19" extent="1-1"/>
+<wire x1="80.2005" y1="6.6245" x2="80.285790625" y2="6.791146875" width="0" layer="19" extent="1-1"/>
 </signal>
 <signal name="SOL1-">
@@
 <wire x1="88.28626875" y1="9.0805" x2="84.582" y2="9.0805" width="0.3048" layer="16"/>
 <wire x1="84.582" y1="9.0805" x2="81.28" y2="5.969" width="0.3048" layer="16"/>
-<via x="71.91481875" y="6.190184375" extent="1-16" drill="0.35"/>
+<via x="69.13481875" y="6.220184375" extent="1-16" drill="0.35"/>
 <wire x1="62.484" y1="11.1125" x2="67.437" y2="6.1595" width="0.3048" layer="1"/>
 <via x="62.484" y="11.1125" extent="1-16" drill="0.35"/>
@@
 <wire x1="75.6539" y1="5.969" x2="75.4304" y2="6.223" width="0.3048" layer="16"/>
 <wire x1="75.4304" y1="6.223" x2="74.9097" y2="6.78815" width="0.3048" layer="16"/>
-<wire x1="74.9097" y1="6.78815" x2="73.43775" y2="6.78815" width="0.3048" layer="16"/>
-<wire x1="72.821309375" y1="6.173784375" x2="73.43775" y2="6.78815" width="0.3048" layer="16"/>
-<wire x1="71.91481875" y1="6.190184375" x2="72.821309375" y2="6.173784375" width="0.3048" layer="16"/>
+<wire x1="74.9097" y1="6.78815" x2="71.01734375" y2="6.78815" width="0.3048" layer="16"/>
+<wire x1="71.01734375" y1="6.78815" x2="70.501309375" y2="6.27385" width="0.3048" layer="16"/>
+<wire x1="70.501309375" y1="6.27385" x2="70.5003375" y2="6.220184375" width="0.3048" layer="16"/>
+<wire x1="70.5003375" y1="6.220184375" x2="69.13481875" y2="6.220184375" width="0.3048" layer="16"/>
 <wire x1="38.3743" y1="25.2349" x2="58.928" y2="25.2095" width="0.254" layer="16"/>
 <wire x1="59.27725" y1="24.8285" x2="59.28995" y2="21.0312" width="0.3048" layer="1"/>
-<wire x1="67.437" y1="6.1595" x2="71.884134375" y2="6.1595" width="0.3048" layer="1"/>
-<wire x1="71.884134375" y1="6.1595" x2="71.91481875" y2="6.190184375" width="0.3048" layer="1"/>
+<wire x1="67.437" y1="6.1595" x2="69.074134375" y2="6.1595" width="0.3048" layer="1"/>
+<wire x1="69.13481875" y1="6.220184375" x2="69.074134375" y2="6.1595" width="0.3048" layer="1"/>
 </signal>
 <signal name="N$7">
