File: CURRENT/openSX70_ALPHA_V7-20181101.sch (EAGLE design)
At the start: 44 parts, among them J1 687106183722, Q1 5.8A/30V/35mΩ, Q2 5.8A/30V/35mΩ, U1 ATMEGA328P_TQFP, Y1 CSTCE8M00G52Z-R0

Commit message: new all new layout 7.0
Parts:
- removed LED1: (no value), led:LEDCHIPLED_0805
- removed R8: 1K 1/10W, Seeed-Resistor:SMD-RES-1K-5%-1/10W(0603)
Connections:
- removed net N$5: LED1.C, R8.2
- net GND: no longer R8.1
- net LED: no longer LED1.A
Other:
- note removed: "LED (OPTION 1)"
Changed lines of the file:
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@@
 <part name="FRAME1" library="frames" library_urn="urn:adsk.eagle:library:229" deviceset="DINA4_L" device="" value="openSX70 main board"/>
 <part name="SOL1" library="openSX70" deviceset="SX70-SOLENOID1-2PADS" device=""/>
-<part name="LED1" library="led" library_urn="urn:adsk.eagle:library:259" deviceset="LED" device="CHIPLED_0805" package3d_urn="urn:adsk.eagle:package:15821/2"/>
 <part name="U1" library="openSX70" deviceset="ATMEGA328P_TQFP" device="" value="ATMEGA328P_TQFP"/>
 <part name="GND1" library="SparkFun-PowerSymbols" library_urn="urn:adsk.eagle:library:530" deviceset="GND" device=""/>
@@
 <part name="R6" library="Seeed-Resistor" library_urn="urn:adsk.eagle:library:474" deviceset="SMD-RES-10K-1%-1/10W(0603)" device="" package3d_urn="urn:adsk.eagle:package:32791/1" value="10K"/>
 <part name="R7" library="Seeed-Resistor" library_urn="urn:adsk.eagle:library:474" deviceset="SMD-RES-100R-5%-1/10W(0603)" device="" package3d_urn="urn:adsk.eagle:package:32791/1" value="100R"/>
-<part name="R8" library="Seeed-Resistor" library_urn="urn:adsk.eagle:library:474" deviceset="SMD-RES-1K-5%-1/10W(0603)" device="" package3d_urn="urn:adsk.eagle:package:32791/1" value="1K 1/10W"/>
 <part name="GND8" library="SparkFun-PowerSymbols" library_urn="urn:adsk.eagle:library:530" deviceset="GND" device=""/>
 <part name="R9" library="Seeed-Resistor" library_urn="urn:adsk.eagle:library:474" deviceset="SMD-RES-15K-1%-1/10W(0603)" device="" package3d_urn="urn:adsk.eagle:package:32791/1" value="15K 1/10W"/>
@@
 <part name="GND12" library="SparkFun-PowerSymbols" library_urn="urn:adsk.eagle:library:530" deviceset="GND" device=""/>
 <part name="P+5" library="openSX70" deviceset="VCC" device="" value="6V"/>
-<part name="GND16" library="SparkFun-PowerSymbols" library_urn="urn:adsk.eagle:library:530" deviceset="GND" device=""/>
 <part name="C2" library="Seeed-Capacitor" library_urn="urn:adsk.eagle:library:464" deviceset="CERAMIC-100NF-50V-10%-X7R(0603)" device="" package3d_urn="urn:adsk.eagle:package:32378/1" value="100nf"/>
 <part name="C1" library="Seeed-Capacitor" library_urn="urn:adsk.eagle:library:464" deviceset="CERAMIC-10UF-10V-10%-X5R(0603)" device="" package3d_urn="urn:adsk.eagle:package:32378/1" value="10uf"/>
@@
 <text x="93.98" y="22.86" size="2.1844" layer="97" align="center">VOLTAGE
 REGULATOR</text>
-<text x="35.56" y="33.02" size="2.1844" layer="97">LED
-(OPTION 1)</text>
 <text x="0" y="68.58" size="2.1844" layer="97">S8 LIMITER RESISTORS TO 3.3V</text>
 <text x="50.8" y="68.58" size="2.1844" layer="97">S9 LIMITER RESISTORS TO 3.3V</text>
@@
 <text x="215.9" y="63.5" size="1.778" layer="95">S4B</text>
 <text x="221.742" y="59.436" size="1.778" layer="97" align="center">PRE-ALPHA</text>
-<text x="35.56" y="33.02" size="2.1844" layer="97">LED
-(OPTION 1)</text>
 <text x="0" y="40.64" size="2.1844" layer="97">LED
 (OPTION 2)</text>
@@
 </instance>
 <instance part="SOL1" gate="G$1" x="220.98" y="40.64" rot="R180"/>
-<instance part="LED1" gate="G$1" x="40.64" y="20.32">
-<attribute name="NAME" x="44.196" y="15.748" size="1.778" layer="95" rot="R90"/>
-<attribute name="VALUE" x="46.355" y="15.748" size="1.778" layer="96" rot="R90"/>
-</instance>
 <instance part="U1" gate="U$1" x="170.18" y="96.52">
 <attribute name="NAME" x="149.86" y="130.302" size="1.778" layer="95"/>
@@
 <attribute name="VALUE" x="208.28" y="119.38" size="1.27" layer="96" ratio="10"/>
 </instance>
-<instance part="R8" gate="G$1" x="40.64" y="10.16" rot="R90">
-<attribute name="NAME" x="39.37" y="6.35" size="1.27" layer="95" ratio="10" rot="R90"/>
-<attribute name="VALUE" x="43.18" y="6.35" size="1.27" layer="96" ratio="10" rot="R90"/>
-</instance>
 <instance part="GND8" gate="1" x="88.9" y="63.5" rot="R90">
 <attribute name="VALUE" x="89.154" y="63.5" size="1.778" layer="96" rot="R90" align="top-center"/>
@@
 <instance part="P+5" gate="VCC" x="167.64" y="147.32" rot="R90">
 <attribute name="VALUE" x="170.18" y="144.78" size="1.778" layer="96" rot="R180"/>
-</instance>
-<instance part="GND16" gate="1" x="40.64" y="5.08">
-<attribute name="VALUE" x="40.64" y="4.826" size="1.778" layer="96" align="top-center"/>
 </instance>
 <instance part="C2" gate="G$1" x="93.98" y="9.144" rot="R270">
@@
 <wire x1="193.04" y1="68.58" x2="205.74" y2="68.58" width="0.1524" layer="91"/>
 <label x="195.58" y="68.58" size="1.778" layer="95"/>
-</segment>
-<segment>
-<pinref part="LED1" gate="G$1" pin="A"/>
-<wire x1="40.64" y1="22.86" x2="40.64" y2="30.48" width="0.1524" layer="91"/>
-<label x="45.72" y="27.94" size="1.778" layer="95"/>
 </segment>
 <segment>
@@
 <wire x1="238.76" y1="139.7" x2="238.76" y2="137.16" width="0.1524" layer="91"/>
 <junction x="238.76" y="139.7"/>
-</segment>
-<segment>
-<pinref part="R8" gate="G$1" pin="1"/>
-<pinref part="GND16" gate="1" pin="GND"/>
-<wire x1="40.64" y1="7.62" x2="40.64" y2="6.35" width="0.1524" layer="91"/>
 </segment>
 <segment>
@@
 </segment>
 </net>
-<net name="N$5" class="0">
-<segment>
-<pinref part="R8" gate="G$1" pin="2"/>
-<pinref part="LED1" gate="G$1" pin="C"/>
-<wire x1="40.64" y1="15.24" x2="40.64" y2="13.97" width="0.1524" layer="91"/>
-<wire x1="40.64" y1="12.7" x2="40.64" y2="13.97" width="0.1524" layer="91"/>
-<junction x="40.64" y="13.97"/>
-</segment>
-</net>
