File: CURRENT/openSX70_ALPHA_V7-20181101.brd (EAGLE design)
At the start: 95.9 x 27.9 mm, 44 parts, among them J1 687106183722, Q1 5.8A/30V/35mΩ, Q2 5.8A/30V/35mΩ, U1 ATMEGA328P_TQFP, Y1 CSTCE8M00G52Z-R0

Commit message: new all new layout 7.0
Parts:
- removed LED1: (no value), led:CHIPLED_0805
- removed R8: 1K 1/10W, Seeed-Resistor:R0603
- moved R10 23.7 mm to (10.4, 4.41)
- moved R6 19.6 mm to (12.2, 2.53)
- moved R9 17.9 mm to (16.3, 4.38)
- moved R5 14.6 mm to (16.9, 2.57)
- moved R7 12.7 mm to (97.0, 16.9), turned to 0 degrees
- moved C2 5.00 mm to (14.0, 12.3)
- moved R14 4.61 mm to (19.4, 20.4)
- moved R12 3.54 mm to (67.6, 23.5)
- moved R11 3.16 mm to (17.8, 18.4)
- moved R16 3.16 mm to (27.6, 22.7)
- moved R15 2.24 mm to (16.8, 16.4)
- moved C3 2.16 mm to (14.3, 19.0), turned to 0 degrees
- moved C1 1.50 mm to (14.0, 8.06)
- moved R4 0.71 mm to (72.7, 23.3)
- moved LD11172.5V 0.50 mm to (7.12, 10.2)
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Connections:
- removed net N$5: LED1.C, R8.2
- net GND: no longer R8.1
- net LED: no longer LED1.A
Routing:
- net LED: track 137.7 -> 0.00 mm, vias 7 -> 0
- net RXD: track 107.3 -> 0.00 mm, vias 2 -> 0
- net S8@6V: track 101.6 -> 0.00 mm, vias 4 -> 0
- net DTR: track 95.3 -> 0.00 mm, vias 4 -> 0
- net S9@6V: track 93.5 -> 0.00 mm, vias 4 -> 0
- net V1: track 84.6 -> 0.00 mm, vias 6 -> 0
- net LED2: track 83.2 -> 0.00 mm
- net TXD: track 82.9 -> 0.00 mm, vias 4 -> 0
- net PDIODE: track 81.2 -> 0.00 mm, vias 5 -> 0
- net V2-SDA: track 81.0 -> 0.00 mm, vias 2 -> 0
- net V3-SCL: track 79.4 -> 0.00 mm, vias 8 -> 0
- net S1: track 79.3 -> 0.00 mm, vias 5 -> 0
- net S2: track 78.1 -> 0.00 mm, vias 4 -> 0
- net SOL2: track 77.2 -> 0.00 mm, vias 4 -> 0
- net S9@2.5V: track 76.7 -> 0.00 mm, vias 4 -> 0
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Other:
- board text added: "20181101"
- board text added: "layout 7.0"
- board text added: "openSX70 project visit www.openSX70.com version 7.0 "ALPHA" 20181101 by Joaquín de Prada"
- board text removed: "20181015"
- board text removed: "VCC IN SEL"
- board text removed: "layout 6.5"
- board text removed: "openSX70 project visit www.openSX70.com version 6.5 "ALPHA" 20181015 by Joaquín de Prada"

Commit message: v7 probably abandoned
Parts:
- moved R16 2.12 mm to (29.1, 24.2)
- moved R12 0.51 mm to (67.4, 23.0), turned to 0 degrees
Routing:
- net 3.3V: track 102.9 -> 119.6 mm, vias 2 -> 3
- net SOL1: track 0.00 -> 10.2 mm
- net RST: track 0.00 -> 6.96 mm
- net N$3: track 0.00 -> 6.90 mm
- net N$1: track 0.00 -> 5.68 mm
- net N$9: track 0.00 -> 2.37 mm
- net GND: track 0.00 -> 2.09 mm
