File: CURRENT/openSX70_ALPHA_V6-2-1-20181102.brd (EAGLE design)
At the start: 95.9 x 27.9 mm, 39 parts, among them J1 687106183722, Q1 5.8A/30V/35mΩ, Q2 5.8A/30V/35mΩ, U1 ATMEGA328P_TQFP, Y1 CSTCE8M00G52Z-R0

Commit message: working on 6.2.2
Routing:
- net RST: track 66.0 -> 84.3 mm
- net FF: track 69.3 -> 68.3 mm
- net SOL2: track 85.7 -> 84.9 mm

Commit message: 6.2.1 WIP
Parts:
- moved C1 4.99 mm to (11.2, 5.56)
- moved R3 0.51 mm to (70.0, 23.2)
- moved R4 0.48 mm to (72.3, 23.3)
Connections:
- removed net SCL: U1.28
- removed net SDA: U1.27
- net LED2: now also U1.9
- net V1: now also U1.22
- net V2-SDA: now also U1.27
- net V3-SCL: now also U1.28
Routing:
- net V2-SDA: track 0.00 -> 86.2 mm, vias 0 -> 2
- net PDIODE: track 12.3 -> 96.2 mm, vias 1 -> 5
- net V1: track 0.00 -> 82.9 mm, vias 0 -> 4
- net V3-SCL: track 0.00 -> 78.6 mm, vias 0 -> 2
- net LED2: track 0.00 -> 65.2 mm, vias 0 -> 4
- net S2: track 23.6 -> 81.9 mm, vias 2 -> 4
- net LED: track 78.0 -> 100.8 mm, vias 2 -> 3
- net S9@6V: track 89.9 -> 95.3 mm
- net TXD: track 85.7 -> 88.1 mm
- net S9@2.5V: track 73.4 -> 75.3 mm
- net SOL2: track 84.9 -> 83.0 mm
- net RST: track 84.3 -> 82.7 mm, vias 2 -> 0
- net 3.3V: track 132.7 -> 134.0 mm
- net 6V: track 184.5 -> 185.8 mm
- net S8@2.5V: track 67.7 -> 68.8 mm
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