File: CURRENT/openSX70_ALPHA_V6-2-2-20181103.brd (EAGLE design)
At the start: 95.9 x 27.9 mm, 39 parts, among them J1 687106183722, Q1 5.8A/30V/35mΩ, Q2 5.8A/30V/35mΩ, U1 ATMEGA328P_TQFP, Y1 CSTCE8M00G52Z-R0

Commit message: new board ready for manufacturing 6.2.2
Parts:
- moved C2 2.92 mm to (16.1, 12.4)
Routing:
- net 6V: track 185.2 -> 179.8 mm
- net N$3: track 6.94 -> 9.90 mm
- net S9@6V: track 95.3 -> 97.6 mm
- net LED2: track 65.1 -> 63.1 mm
- net PDIODE: track 95.6 -> 97.3 mm
- net GND: track 0.08 -> 1.63 mm, vias 0 -> 20
- net FF: track 65.9 -> 67.1 mm
- net S8@6V: track 87.1 -> 88.4 mm
- net SOL1: track 9.93 -> 11.2 mm
- net V1: track 82.6 -> 81.5 mm
- net S5: track 15.8 -> 15.0 mm
- net DTR: track 106.9 -> 106.2 mm
- net N$4: track 5.81 -> 6.43 mm
- net S1: track 80.5 -> 79.9 mm, vias 5 -> 3
Other:
- board text added: "1W"
- board text added: "20181103"
- board text added: "openSX70 project visit www.openSX70.com version 6.2.2 "ALPHA" 20181103 by Joaquín de Prada"
- board text removed: "20181102"
- board text removed: "openSX70 project visit www.openSX70.com version 6.2.2 "ALPHA" 20181102 by Joaquín de Prada"

Commit message: new layout minor changes
Parts:
- moved C6 0.57 mm to (71.6, 17.1)
Routing:
- net V2-SDA: track 86.1 -> 78.6 mm
- net V3-SCL: track 78.8 -> 76.2 mm
- net GND: track 1.63 -> 3.70 mm
- net PDIODE: track 97.3 -> 95.9 mm
- removed copper zone on layer 1, net N$11
- removed copper zone on layer 1, net N$12
- removed copper zone on layer 1, net N$13
- removed copper zone on layer 1, net N$14
- removed copper zone on layer 1, net N$16
- removed copper zone on layer 16, net N$18
- removed copper zone on layer 1, net N$7
- removed copper zone on layer 1, net N$8
