File: CURRENT/openSX70_ALPHA_V6-2-3-20181104.brd (EAGLE design)
At the start: 95.9 x 27.9 mm, 39 parts, among them J1 687106183722, Q1 5.8A/30V/35mΩ, Q2 5.8A/30V/35mΩ, U1 ATMEGA328P_TQFP, Y1 CSTCE8M00G52Z-R0

Commit message: changed connector S-pad on 6.2.3
Parts:
- U$1: device openSX70:SX70-7-PAD -> _openSX70:SX70-7-PAD-PROPER
- moved U$1 7.15 mm to (89.2, 17.3), turned to 296 degrees
- moved C7 0.26 mm to (69.8, 19.6)
Connections:
- net 6V: now also U$1.VCC; no longer U$1.VCC-6V
- net MOTOR-HEADER: now also U$1.MOTOR; no longer U$1.MOTOR+
Routing:
- net N$3: track 9.53 -> 7.18 mm
- net N$4: track 6.43 -> 5.69 mm
- net S9@2.5V: track 75.2 -> 74.6 mm
- net GND: vias 20 -> 21
Other:
- board text added: "20181104"
- board text added: "C"
- board text added: "LM"
- board text added: "layout 6.2.3"
- board text added: "openSX70 project visit www.openSX70.com version 6.2.3 "ALPHA" 20181104 by Joaquín de Prada"
- board text removed: "20181103"
- board text removed: "K"
- board text removed: "layout 6.2.2"
- board text removed: "openSX70 project visit www.openSX70.com version 6.2.2 "ALPHA" 20181103 by Joaquín de Prada"
