File: CURRENT/openSX70_ALPHA_V6-2-4-20181127.brd (EAGLE design)
At the start: 95.9 x 27.9 mm, 39 parts, among them J1 687106183722, Q1 5.8A/30V/35mΩ, Q2 5.8A/30V/35mΩ, U1 ATMEGA328P_TQFP, Y1 CSTCE8M00G52Z-R0

Commit message: new LED footprint!
Parts:
- removed R16: 1K 1/10W, Seeed-Resistor:R0603
- removed U$3: DUAL-LED-0603-BIS, _openSX70:LED_APHB1608SYKSURKC
- added R13: 15K 1/10W, Seeed-Resistor:R0603
- added U$4: LTST-C195KGJRKT, LTST-C195KGJRKT:LTST-BILED-15X16
- R11: value 15K 1/10W -> 1K 1/10W
- moved R11 18.7 mm to (32.9, 27.9), turned to 270 degrees
Connections:
- removed net N$9: R16.2, U$3.2, U$3.4
- new net N$2: R11.2, U$4.P$3, U$4.P$4
- net GND: now also R11.1; no longer R16.1
- net LED: now also U$4.P$1; no longer U$3.1
- net LED2: now also U$4.P$2; no longer U$3.3
- net PDIODE: now also R13.2; no longer R11.2
- net V3-SCL: now also R13.1; no longer R11.1
Routing:
- net N$2: track 0.00 -> 2.68 mm
- net N$9: track 2.61 -> 0.00 mm
- net LED2: track 63.1 -> 60.5 mm
- net LED: track 101.1 -> 99.9 mm
- net S8@6V: track 88.2 -> 87.6 mm
Other:
- outline, holes or cut-outs redrawn
- board text added: "20181128"
- board text added: "openSX70 project visit www.openSX70.com version 6.2.4 "ALPHA" 20181128 by Joaquín de Prada"
- board text removed: "20181127"
- board text removed: "openSX70 project visit www.openSX70.com version 6.2.4 "ALPHA" 20181104 by Joaquín de Prada"
