File: CURRENT/openSX70_ALPHA_V6-2-4-20181127.sch (EAGLE design)
At the start: 39 parts, among them J1 687106183722, Q1 5.8A/30V/35mΩ, Q2 5.8A/30V/35mΩ, U1 ATMEGA328P_TQFP, Y1 CSTCE8M00G52Z-R0

Commit message: new LED footprint!
Parts:
- removed R16: 1K 1/10W, Seeed-Resistor:SMD-RES-1K-5%-1/10W(0603)
- removed U$3: DUAL-LED-0603-BIS, _openSX70:DUAL-LED-0603-BIS
- added R13: 15K 1/10W, Seeed-Resistor:SMD-RES-15K-1%-1/10W(0603)
- added U$4: LTST-C195KGJRKT, LTST-C195KGJRKT:LTST-C195KGJRKT
- R11: value 15K 1/10W -> 1K 1/10W; device Seeed-Resistor:SMD-RES-15K-1%-1/10W(0603) -> Seeed-Resistor:SMD-RES-1K-5%-1/10W(0603)
Connections:
- removed net N$9: R16.2, U$3.C, U$3.C1
- new net N$2: R11.2, U$4.K1, U$4.K2
- net GND: now also R11.1; no longer R16.1
- net LED: now also U$4.A1; no longer U$3.A
- net LED2: now also U$4.A2; no longer U$3.A1
- net PDIODE: now also R13.2; no longer R11.2
- net V3-SCL: now also R13.1; no longer R11.1
Other:
- note added: "A"
- note added: "C"
- note added: "v 6.2.4"
- note removed: "v 6.6.3"
- moved on the sheet: R11
