File: CURRENT/openSX70_ALPHA_V6-2-5-20181220.brd (EAGLE design)
At the start: 95.9 x 27.9 mm, 39 parts, among them J1 687106183722, Q1 5.8A/30V/35mΩ, Q2 5.8A/30V/35mΩ, U1 ATMEGA328P_TQFP, Y1 CSTCE8M00G52Z-R0

Commit message: new main PCB fixed 3rd resistor on Photodiode!
Parts:
- added TP1: TEST-POINT3X4, SparkFun-Connectors:PAD.03X.04
- moved U$4 0.08 mm to (30.2, 27.2)
Connections:
- new net N$5: TP1.P$1, U$2.FT
Routing:
- net N$5: track 0.00 -> 1.93 mm
- net PDIODE: track 95.9 -> 94.0 mm
- net GND: track 3.70 -> 2.44 mm, vias 25 -> 22
- net 3.3V: track 133.6 -> 132.6 mm
- net S8@2.5V: track 68.7 -> 67.9 mm
- net S3: track 13.0 -> 13.7 mm
- net 6V: track 179.7 -> 179.1 mm
Other:
- board text added: ""ALPHA-2""
- board text added: "TP-FT"
- board text added: "openSX70 project visit www.openSX70.com version 6.2.5"ALPHA-2" 20181220 by Joaquín de Prada"
- board text removed: ""ALPHA""
- board text removed: "FT"
- board text removed: "openSX70 project visit www.openSX70.com version 6.2.5"ALPHA" 20181220 by Joaquín de Prada"
