File: CURRENT/openSX70_ALPHA-2B_V6-2-6-20190105-S2-22.brd (EAGLE design)
At the start: 95.9 x 27.9 mm, 40 parts, among them J1 687106183722, Q1 5.8A/30V/35mΩ, Q2 5.8A/30V/35mΩ, U1 ATMEGA328P_TQFP, Y1 CSTCE8M00G52Z-R0

Commit message: gerbers
Connections:
- net S2: now also U1.22; no longer U1.32
Routing:
- net S2: track 81.4 -> 88.3 mm, vias 4 -> 2
- net V1: track 82.7 -> 84.1 mm
- net S8@2.5V: track 67.9 -> 68.7 mm
Other:
- board text added: ""ALPHA-2B""
- board text added: "20190105"
- board text added: "layout 6.2.6S2-22"
- board text added: "openSX70 project visit www.openSX70.com version 6.2.6"ALPHA-2B" 20190105 by Joaquín de Prada"
- board text removed: ""ALPHA"-aFtr8"
- board text removed: "20181220"
- board text removed: "layout 6.2.5"
- board text removed: "openSX70 project visit www.openSX70.com version 6.2.5"ALPHA"-aFtr8 20190111 by Joaquín de Prada"
