File: CURRENT/openSX70_U2_V6-3-1-20190307.brd (EAGLE design)
At the start: 95.9 x 27.9 mm, 39 parts, among them IC1 AD654, J1 687106183722, Q1 5.8A/30V/35mΩ, Q2 5.8A/30V/35mΩ, U1 ATMEGA328P_TQFP, Y1 CSTCE8M00G52Z-R0

Commit message: few changes
Parts:
- moved R8 3.19 mm to (17.2, 14.5)
- moved C3 3.11 mm to (11.8, 14.4), turned to 90 degrees
Routing:
- net RXD: track 108.9 -> 120.9 mm
- net DTR: track 106.0 -> 108.4 mm
- net 6V: track 176.7 -> 178.3 mm
- net 3.3V: track 131.1 -> 132.7 mm
