File: CURRENT/openSX70_MEROE_V7_20190603.brd (EAGLE design)
At the start: 95.9 x 27.9 mm, 42 parts, among them J1 687106183722, Q1 5.8A/30V/35mΩ, Q2 5.8A/30V/35mΩ, U1 ATMEGA328P_TQFP, U2 TPS79501DCQ, Y1 CSTCE8M00G52Z-R0

Commit message: Meröe more or less finished. TCS3200
Parts:
- moved TP2 1.47 mm to (20.5, 10.1)
- moved C4 1.45 mm to (17.8, 10.9)
- moved TP1 0.23 mm to (22.7, 23.4)
Routing:
- net GND: track 2.93 -> 6.15 mm, vias 17 -> 32
- net DTR: track 108.0 -> 111.0 mm
- net RST: track 79.3 -> 82.3 mm
- net TXD: track 84.9 -> 86.9 mm
- net SDA_S2: track 78.0 -> 79.2 mm, vias 1 -> 2
- net S8@2.5V: track 67.9 -> 69.1 mm
- net 3.3V: track 160.7 -> 159.5 mm
- net LM: track 81.7 -> 80.6 mm
- net FF: track 68.1 -> 69.2 mm
- net TCS3200_S1: track 73.0 -> 73.9 mm
- net S9@2.5V: track 74.3 -> 75.2 mm
Other:
- board text added: "3.3V"
