File: CURRENT/openSX70_MEROE_V7-5_20190606.brd (EAGLE design)
At the start: 95.9 x 27.9 mm, 46 parts, among them J1 687106183722, Q1 5.8A/30V/35mΩ, Q2 5.8A/30V/35mΩ, U1 ATMEGA328P_TQFP, U2 TPS79501DCQ, Y1 CSTCE8M00G52Z-R0

Commit message: New Meroë 7.5 with 3 added capacitors. Crowded
Parts:
- moved R4 1.31 mm to (73.5, 23.5)
- moved R3 1.19 mm to (71.7, 23.5)
Routing:
- net SOL2: track 83.5 -> 84.8 mm
- net N$3: track 5.97 -> 4.85 mm
- net SOL1: track 11.9 -> 11.2 mm
- net GND: vias 30 -> 23
Other:
- board text added: "20190606"
- board text added: "MEROË"
- board text added: "layout 7.5"
- board text added: "openSX70 project visit www.openSX70.com version 7.5E "MEROË" 20190506 by Joaquín de Prada"
- board text removed: "20190603"
- board text removed: "MERÖE"
- board text removed: "openSX70 project visit www.openSX70.com version 7 "MEROE" 20190503 by Joaquín de Prada"
