File: CURRENT/EDWIN_TSL237T/openSX70_MEROEC_V7-9C_20200625-TCS3200.sch (EAGLE design)
At the start: 44 parts, among them J1 687106183722, Q1 5.8A/30V/35mΩ, Q2 5.8A/30V/35mΩ, U1 ATMEGA328P_TQFP, U2 TPS79501DCQ, Y1 CSTCE8M00G52Z-R0

Commit message: Latest
Parts:
- removed U$3: TSL237T, _openSX70:TSL237T
- added S0: S0, SparkFun-Jumpers:JUMPER-SMT_3_1-NC_TRACE_SILK
- added S2: S2, SparkFun-Jumpers:JUMPER-SMT_3_1-NC_TRACE_SILK
- added TP4: TEST-POINT3X4, SparkFun-Connectors:TEST-POINT3X4
- added U3: TCS3200D, TCS3200D:TCS3200D
- R5, R9: value 12K 1/10W -> 15K 1/10W
- U$2: device openSX70:SX70-FFA-PAD -> _openSX70:SX70-FFA-PAD
- renumbered Y1 to X1
Connections:
- removed net OE: U$3.OE, U1.PB1(OC1A)
- new net N$7: S0.2, U3.S0
- new net N$8: S2.2, U3.S2
- new net TCS3200_OE: U1.PB1(OC1A), U3.OE
- new net TCS3200_S1: U1.PD2(INT0), U3.S1
- new net TCS3200_S3: U1.PD6(AIN0), U3.S3
- net 3.3V: now also S0.3, S2.3, U3.VDD; no longer U$3.V+
- net GND: now also S0.1, S2.1, U3.GND; no longer U$3.GND
- net LM: now also U3.OUT; no longer U$3.OUT
- net S1: now also TP4.1
Other:
- note added: ""MEROË-C" version"
- note added: "MISO"
- note added: "RESET"
- note added: "SCK"
- note added: "v7.5"
- note removed: ""EDWIN" (MEROË2) version"
- note removed: "v7.7"
- moved on the sheet: C3, R8
